File: Kicad/Cargador.sch (KiCad schematic (older format))
At the start: 0 parts

Commit message: Hicimos el esquemático del cargador, y agregamos la hoja de datos
Parts:
- added C? (x2): CP, symbol CP
- added D?: LED, symbol LED
- added P?: USB_A, symbol USB_A
- added R? (x2): R, symbol R
- added U?: MCP73831, symbol MCP73831
Connections:
- net labels added: +BATT, -BATT
- wire segments 0 -> 17
Changed lines of the file:
@@
 LIBS:device
 LIBS:Gajda_amplif
-LIBS:opa4243
 LIBS:tlc2274
 LIBS:power
@@
 LIBS:bat
 LIBS:batn
-LIBS:microchip
-LIBS:nordicsemi
-LIBS:Power_Management
-LIBS:powerint
-LIBS:references
-LIBS:rfcom
-LIBS:texas
+LIBS:MCP73831
 LIBS:EMG-cache
-EELAYER 25 0
+EELAYER 27 0
 EELAYER END
 $Descr A4 11693 8268
@@
 Sheet 7 7
 Title ""
-Date ""
+Date "19 sep 2016"
 Rev ""
 Comp ""
@@
 Comment4 ""
 $EndDescr
+$Comp
+L MCP73831 U?
+U 1 1 57E06106
+P 5250 3050
+F 0 "U?" H 5250 2900 60  0000 C CNN
+F 1 "MCP73831" H 5250 3600 60  0000 C CNN
+F 2 "" H 5250 3600 60  0000 C CNN
+F 3 "" H 5250 3600 60  0000 C CNN
+	1    5250 3050
+	-1   0    0    1
+$EndComp
+$Comp
+L CP C?
+U 1 1 57E06124
+P 6400 3350
+F 0 "C?" H 6425 3450 50  0000 L CNN
+F 1 "CP" H 6425 3250 50  0000 L CNN
+F 2 "" H 6438 3200 50  0000 C CNN
+F 3 "" H 6400 3350 50  0000 C CNN
+	1    6400 3350
+	1    0    0    -1
+$EndComp
+$Comp
+L CP C?
+U 1 1 57E06133
+P 3900 3250
+F 0 "C?" H 3925 3350 50  0000 L CNN
+F 1 "CP" H 3925 3150 50  0000 L CNN
+F 2 "" H 3938 3100 50  0000 C CNN
+F 3 "" H 3900 3250 50  0000 C CNN
+	1    3900 3250
+	1    0    0    -1
+$EndComp
+$Comp
+L R R?
+U 1 1 57E0616A
+P 6000 3500
+F 0 "R?" V 6080 3500 50  0000 C CNN
+F 1 "R" V 6000 3500 50  0000 C CNN
+F 2 "" V 5930 3500 50  0000 C CNN
+F 3 "" H 6000 3500 50  0000 C CNN
+	1    6000 3500
+	1    0    0    -1
+$EndComp
+$Comp
+L R R?
+U 1 1 57E06179
+P 4450 3550
+F 0 "R?" V 4530 3550 50  0000 C CNN
+F 1 "R" V 4450 3550 50  0000 C CNN
+F 2 "" V 4380 3550 50  0000 C CNN
+F 3 "" H 4450 3550 50  0000 C CNN
+	1    4450 3550
+	0    -1   -1   0
+$EndComp
+$Comp
+L LED D?
+U 1 1 57E06194
+P 4150 3350
+F 0 "D?" H 4150 3450 50  0000 C CNN
+F 1 "LED" H 4150 3250 50  0000 C CNN
+F 2 "" H 4150 3350 50  0000 C CNN
+F 3 "" H 4150 3350 50  0000 C CNN
+	1    4150 3350
+	0    -1   -1   0
+$EndComp
+$Comp
+L -BATT #PWR?
+U 1 1 57E06258
+P 3900 3750
+F 0 "#PWR?" H 3900 3600 50  0001 C CNN
+F 1 "-BATT" H 3900 3890 50  0000 C CNN
+F 2 "" H 3900 3750 50  0000 C CNN
+F 3 "" H 3900 3750 50  0000 C CNN
+	1    3900 3750
+	-1   0    0    1
+$EndComp
+$Comp
+L -BATT #PWR?
+U 1 1 57E0628F
+P 6000 3800
+F 0 "#PWR?" H 6000 3650 50  0001 C CNN
+F 1 "-BATT" H 6000 3940 50  0000 C CNN
+F 2 "" H 6000 3800 50  0000 C CNN
+F 3 "" H 6000 3800 50  0000 C CNN
+	1    6000 3800
+	-1   0    0    1
+$EndComp
+Wire Wire Line
+	4600 3550 4750 3550
+Wire Wire Line
+	4750 3550 4750 3400
+Wire Wire Line
+	4300 3550 4150 3550
+Wire Wire Line
+	4150 3150 4150 3100
+Wire Wire Line
+	3400 3100 4750 3100
+Connection ~ 4150 3100
+Wire Wire Line
+	3900 3400 3900 3750
+Wire Wire Line
+	5700 3250 6000 3250
+Wire Wire Line
+	6000 3250 6000 3350
+Wire Wire Line
+	6000 3800 6000 3650
+Wire Wire Line
+	5700 3400 5700 3750
+Wire Wire Line
+	5700 3750 6400 3750
+Connection ~ 6000 3750
+Wire Wire Line
+	5700 3100 6900 3100
+Wire Wire Line
+	6400 3100 6400 3200
+Wire Wire Line
+	6400 3750 6400 3500
+$Comp
+L +BATT #PWR?
+U 1 1 57E062FB
+P 6900 3050
+F 0 "#PWR?" H 6900 2900 50  0001 C CNN
+F 1 "+BATT" H 6900 3190 50  0000 C CNN
+F 2 "" H 6900 3050 50  0000 C CNN
+F 3 "" H 6900 3050 50  0000 C CNN
+	1    6900 3050
+	1    0    0    -1
+$EndComp
+Wire Wire Line
+	6900 3100 6900 3050
+Connection ~ 6400 3100
+$Comp
+L USB_A P?
+U 1 1 57E06354
+P 3100 3300
+F 0 "P?" H 3300 3100 50  0000 C CNN
+F 1 "USB_A" H 3050 3500 50  0000 C CNN
+F 2 "" V 3050 3200 50  0000 C CNN
+F 3 "" V 3050 3200 50  0000 C CNN
+	1    3100 3300
+	0    -1   1    0
+$EndComp
+Connection ~ 3900 3100
+Wire Wire Line
+	3400 3400 3400 3700
+Wire Wire Line
+	3400 3700 3900 3700
+Connection ~ 3900 3700
 $EndSCHEMATC

Commit message: Agregado componente DC/DC
Parts:
- gave numbers to parts that had none: 7
Changed lines of the file:
@@
 LIBS:batn
 LIBS:MCP73831
+LIBS:maxim
+LIBS:max8881
 LIBS:EMG-cache
-EELAYER 27 0
+EELAYER 25 0
 EELAYER END
 $Descr A4 11693 8268
@@
 $EndDescr
 $Comp
-L MCP73831 U?
+L MCP73831 U4
 U 1 1 57E06106
 P 5250 3050
-F 0 "U?" H 5250 2900 60  0000 C CNN
+F 0 "U4" H 5250 2900 60  0000 C CNN
 F 1 "MCP73831" H 5250 3600 60  0000 C CNN
 F 2 "" H 5250 3600 60  0000 C CNN
@@
 $EndComp
 $Comp
-L CP C?
+L CP C8
 U 1 1 57E06124
 P 6400 3350
-F 0 "C?" H 6425 3450 50  0000 L CNN
+F 0 "C8" H 6425 3450 50  0000 L CNN
 F 1 "CP" H 6425 3250 50  0000 L CNN
 F 2 "" H 6438 3200 50  0000 C CNN
@@
 $EndComp
 $Comp
-L CP C?
+L CP C7
 U 1 1 57E06133
 P 3900 3250
-F 0 "C?" H 3925 3350 50  0000 L CNN
+F 0 "C7" H 3925 3350 50  0000 L CNN
 F 1 "CP" H 3925 3150 50  0000 L CNN
 F 2 "" H 3938 3100 50  0000 C CNN
@@
 $EndComp
 $Comp
-L R R?
+L R R22
 U 1 1 57E0616A
 P 6000 3500
-F 0 "R?" V 6080 3500 50  0000 C CNN
+F 0 "R22" V 6080 3500 50  0000 C CNN
 F 1 "R" V 6000 3500 50  0000 C CNN
 F 2 "" V 5930 3500 50  0000 C CNN
@@
 $EndComp
 $Comp
-L R R?
+L R R21
 U 1 1 57E06179
 P 4450 3550
-F 0 "R?" V 4530 3550 50  0000 C CNN
+F 0 "R21" V 4530 3550 50  0000 C CNN
 F 1 "R" V 4450 3550 50  0000 C CNN
 F 2 "" V 4380 3550 50  0000 C CNN
@@
 $EndComp
 $Comp
-L LED D?
+L LED D1
 U 1 1 57E06194
 P 4150 3350
-F 0 "D?" H 4150 3450 50  0000 C CNN
+F 0 "D1" H 4150 3450 50  0000 C CNN
 F 1 "LED" H 4150 3250 50  0000 C CNN
 F 2 "" H 4150 3350 50  0000 C CNN
@@
 $EndComp
 $Comp
-L -BATT #PWR?
+L -BATT #PWR15
 U 1 1 57E06258
 P 3900 3750
-F 0 "#PWR?" H 3900 3600 50  0001 C CNN
+F 0 "#PWR15" H 3900 3600 50  0001 C CNN
 F 1 "-BATT" H 3900 3890 50  0000 C CNN
 F 2 "" H 3900 3750 50  0000 C CNN
@@
 $EndComp
 $Comp
-L -BATT #PWR?
+L -BATT #PWR16
 U 1 1 57E0628F
 P 6000 3800
-F 0 "#PWR?" H 6000 3650 50  0001 C CNN
+F 0 "#PWR16" H 6000 3650 50  0001 C CNN
 F 1 "-BATT" H 6000 3940 50  0000 C CNN
 F 2 "" H 6000 3800 50  0000 C CNN
@@
 	6400 3750 6400 3500
 $Comp
-L +BATT #PWR?
+L +BATT #PWR17
 U 1 1 57E062FB
 P 6900 3050
-F 0 "#PWR?" H 6900 2900 50  0001 C CNN
+F 0 "#PWR17" H 6900 2900 50  0001 C CNN
 F 1 "+BATT" H 6900 3190 50  0000 C CNN
 F 2 "" H 6900 3050 50  0000 C CNN
@@
 Connection ~ 6400 3100
 $Comp
-L USB_A P?
+L USB_A P3
 U 1 1 57E06354
 P 3100 3300
-F 0 "P?" H 3300 3100 50  0000 C CNN
+F 0 "P3" H 3300 3100 50  0000 C CNN
 F 1 "USB_A" H 3050 3500 50  0000 C CNN
 F 2 "" V 3050 3200 50  0000 C CNN

Commit message: Circuito de cargador modificado. A los demás les agregué capacitor en la alimentación, pines sin conexión y cambié BATT- por GND
Connections:
- net labels added: GND
- net labels removed: -BATT
- wire segments 17 -> 12
- no-connect marks 0 -> 3
Other:
- moved on the sheet: R22
Changed lines of the file:
@@
 L R R22
 U 1 1 57E0616A
-P 6000 3500
-F 0 "R22" V 6080 3500 50  0000 C CNN
-F 1 "R" V 6000 3500 50  0000 C CNN
-F 2 "" V 5930 3500 50  0000 C CNN
-F 3 "" H 6000 3500 50  0000 C CNN
-	1    6000 3500
+P 6000 3400
+F 0 "R22" V 6080 3400 50  0000 C CNN
+F 1 "R" V 6000 3400 50  0000 C CNN
+F 2 "" V 5930 3400 50  0000 C CNN
+F 3 "" H 6000 3400 50  0000 C CNN
+	1    6000 3400
 	1    0    0    -1
 $EndComp
@@
 	0    -1   -1   0
 $EndComp
-$Comp
-L -BATT #PWR15
-U 1 1 57E06258
-P 3900 3750
-F 0 "#PWR15" H 3900 3600 50  0001 C CNN
-F 1 "-BATT" H 3900 3890 50  0000 C CNN
-F 2 "" H 3900 3750 50  0000 C CNN
-F 3 "" H 3900 3750 50  0000 C CNN
-	1    3900 3750
-	-1   0    0    1
-$EndComp
-$Comp
-L -BATT #PWR16
-U 1 1 57E0628F
-P 6000 3800
-F 0 "#PWR16" H 6000 3650 50  0001 C CNN
-F 1 "-BATT" H 6000 3940 50  0000 C CNN
-F 2 "" H 6000 3800 50  0000 C CNN
-F 3 "" H 6000 3800 50  0000 C CNN
-	1    6000 3800
-	-1   0    0    1
-$EndComp
 Wire Wire Line
 	4600 3550 4750 3550
@@
 Connection ~ 4150 3100
 Wire Wire Line
-	3900 3400 3900 3750
-Wire Wire Line
 	5700 3250 6000 3250
-Wire Wire Line
-	6000 3250 6000 3350
-Wire Wire Line
-	6000 3800 6000 3650
-Wire Wire Line
-	5700 3400 5700 3750
-Wire Wire Line
-	5700 3750 6400 3750
-Connection ~ 6000 3750
-Wire Wire Line
-	5700 3100 6900 3100
-Wire Wire Line
-	6400 3100 6400 3200
-Wire Wire Line
-	6400 3750 6400 3500
 $Comp
-L +BATT #PWR17
+L +BATT #PWR24
 U 1 1 57E062FB
-P 6900 3050
-F 0 "#PWR17" H 6900 2900 50  0001 C CNN
-F 1 "+BATT" H 6900 3190 50  0000 C CNN
-F 2 "" H 6900 3050 50  0000 C CNN
-F 3 "" H 6900 3050 50  0000 C CNN
-	1    6900 3050
+P 6400 3100
+F 0 "#PWR24" H 6400 2950 50  0001 C CNN
+F 1 "+BATT" H 6400 3240 50  0000 C CNN
+F 2 "" H 6400 3100 50  0000 C CNN
+F 3 "" H 6400 3100 50  0000 C CNN
+	1    6400 3100
 	1    0    0    -1
 $EndComp
-Wire Wire Line
-	6900 3100 6900 3050
-Connection ~ 6400 3100
 $Comp
 L USB_A P3
@@
 $EndComp
 Connection ~ 3900 3100
+$Comp
+L GND #PWR22
+U 1 1 57FAD4CF
+P 3900 3400
+F 0 "#PWR22" H 3900 3150 50  0001 C CNN
+F 1 "GND" H 3900 3250 50  0000 C CNN
+F 2 "" H 3900 3400 50  0000 C CNN
+F 3 "" H 3900 3400 50  0000 C CNN
+	1    3900 3400
+	1    0    0    -1
+$EndComp
+$Comp
+L GND #PWR23
+U 1 1 57FAD4F1
+P 6000 3550
+F 0 "#PWR23" H 6000 3300 50  0001 C CNN
+F 1 "GND" H 6000 3400 50  0000 C CNN
+F 2 "" H 6000 3550 50  0000 C CNN
+F 3 "" H 6000 3550 50  0000 C CNN
+	1    6000 3550
+	1    0    0    -1
+$EndComp
 Wire Wire Line
-	3400 3400 3400 3700
+	3400 3400 3900 3400
 Wire Wire Line
-	3400 3700 3900 3700
-Connection ~ 3900 3700
+	5700 3400 5700 3550
+Wire Wire Line
+	5700 3550 6400 3550
+Wire Wire Line
+	6400 3550 6400 3500
+Connection ~ 6000 3550
+Wire Wire Line
+	5700 3100 6400 3100
+Wire Wire Line
+	6400 3100 6400 3200
+NoConn ~ 3400 3200
+NoConn ~ 3400 3300
+NoConn ~ 3000 3600
 $EndSCHEMATC

Commit message: Agregados los wrl y wings del amplificador y el cargador.
Parts:
- U4: footprint (none) -> EMG:sot23-5
Changed lines of the file:
@@
 F 0 "U4" H 5250 2900 60  0000 C CNN
 F 1 "MCP73831" H 5250 3600 60  0000 C CNN
-F 2 "" H 5250 3600 60  0001 C CNN
+F 2 "EMG:sot23-5" H 5250 3600 60  0001 C CNN
 F 3 "" H 5250 3600 60  0000 C CNN
 	1    5250 3050

Commit message: Agregados footprints de C_0805 y R_0805 y asociados a resistencias y capacitores del esquemático
Parts:
- C7, C8: footprint (none) -> EMG:C_0805
- R21, R22: footprint (none) -> EMG:R_0805
Changed lines of the file:
@@
 F 0 "C8" H 6425 3450 50  0000 L CNN
 F 1 "CP" H 6425 3250 50  0000 L CNN
-F 2 "" H 6438 3200 50  0001 C CNN
+F 2 "EMG:C_0805" H 6438 3200 50  0001 C CNN
 F 3 "" H 6400 3350 50  0000 C CNN
 	1    6400 3350
@@
 F 0 "C7" H 3925 3350 50  0000 L CNN
 F 1 "CP" H 3925 3150 50  0000 L CNN
-F 2 "" H 3938 3100 50  0001 C CNN
+F 2 "EMG:C_0805" H 3938 3100 50  0001 C CNN
 F 3 "" H 3900 3250 50  0000 C CNN
 	1    3900 3250
@@
 F 0 "R22" V 6080 3400 50  0000 C CNN
 F 1 "R" V 6000 3400 50  0000 C CNN
-F 2 "" V 5930 3400 50  0001 C CNN
+F 2 "EMG:R_0805" V 5930 3400 50  0001 C CNN
 F 3 "" H 6000 3400 50  0000 C CNN
 	1    6000 3400
@@
 F 0 "R21" V 4530 3550 50  0000 C CNN
 F 1 "R" V 4450 3550 50  0000 C CNN
-F 2 "" V 4380 3550 50  0001 C CNN
+F 2 "EMG:R_0805" V 4380 3550 50  0001 C CNN
 F 3 "" H 4450 3550 50  0000 C CNN
 	1    4450 3550
